Commit message: Fixed wrong naming of packages because refactoring

File: mur205_description/urdf/mir_200_v1.urdf.xacro (robot description, xacro)
@@ -4,9 +4,9 @@
   xmlns:sensor="http://playerstage.sourceforge.net/gazebo/xmlschema/#sensor"
   xmlns:xacro="http://ros.org/wiki/xacro">
-  <xacro:include filename="$(find mir_ur5_description)/urdf/include/common_properties.urdf.xacro" />
-  <xacro:include filename="$(find mir_ur5_description)/urdf/include/imu.gazebo.urdf.xacro" />
-  <xacro:include filename="$(find mir_ur5_description)/urdf/include/mir_200.gazebo.xacro" />
-  <xacro:include filename="$(find mir_ur5_description)/urdf/include/mir_200.transmission.xacro" />
-  <xacro:include filename="$(find mir_ur5_description)/urdf/include/sick_s300.urdf.xacro" />
+  <xacro:include filename="$(find mur205_description)/urdf/include/common_properties.urdf.xacro" />
+  <xacro:include filename="$(find mur205_description)/urdf/include/imu.gazebo.urdf.xacro" />
+  <xacro:include filename="$(find mur205_description)/urdf/include/mir_200.gazebo.xacro" />
+  <xacro:include filename="$(find mur205_description)/urdf/include/mir_200.transmission.xacro" />
+  <xacro:include filename="$(find mur205_description)/urdf/include/sick_s300.urdf.xacro" />
   <xacro:property name="deg_to_rad" value="0.017453293" />
   <xacro:property name="mir_200_base_mass" value="58.0" />
@@ -143,5 +143,5 @@
         <origin xyz="${mir_200_act_wheel_dx} 0 0" rpy="${pi/2} 0 ${pi/2}" />
         <geometry>
-          <mesh filename="package://mir_ur5_description/meshes/MiR200_UR5_base_LQ.stl" scale="0.001 0.001 0.001"/> <!--Scale is necessary because stl was generated in mm (correct dimensions) but stl has no measurements and mm are interpreted as m in gazebo-->
+          <mesh filename="package://mur205_description/meshes/MiR200_UR5_base_LQ.stl" scale="0.001 0.001 0.001"/> <!--Scale is necessary because stl was generated in mm (correct dimensions) but stl has no measurements and mm are interpreted as m in gazebo-->
         </geometry>
         <xacro:insert_block name="material_white" />
@@ -150,5 +150,5 @@
         <origin xyz="${mir_200_act_wheel_dx} 0 0" rpy="${pi/2} 0 ${pi/2}" />
         <geometry>
-          <mesh filename="package://mir_ur5_description/meshes/MiR200_UR5_base_LQ.stl" scale="0.001 0.001 0.001"/> <!--Scale is necessary because stl was generated in mm (correct dimensions) but stl has no measurements and mm are interpreted as m in gazebo-->
+          <mesh filename="package://mur205_description/meshes/MiR200_UR5_base_LQ.stl" scale="0.001 0.001 0.001"/> <!--Scale is necessary because stl was generated in mm (correct dimensions) but stl has no measurements and mm are interpreted as m in gazebo-->
         </geometry>
       </collision>

File: mur205_description/urdf/mur205.urdf.xacro (robot description, xacro)
@@ -10,7 +10,7 @@
     <!-- <xacro:property name="robot_name" value='$(arg robot_name)'/> -->
     <!--Include all needed urdf files-->
-    <xacro:include filename="$(find mir_ur5_description)/urdf/mir_200_v1.urdf.xacro"/>
-    <!-- <xacro:include filename="$(find mir_ur5_description)/urdf/ur5.urdf.xacro"/> -->
-    <xacro:include filename="$(find mir_ur5_description)/urdf/ur5_robot.urdf.xacro">
+    <xacro:include filename="$(find mur205_description)/urdf/mir_200_v1.urdf.xacro"/>
+    <!-- <xacro:include filename="$(find mur205_description)/urdf/ur5.urdf.xacro"/> -->
+    <xacro:include filename="$(find mur205_description)/urdf/ur5_robot.urdf.xacro">
         <arg name="tf_prefix" value="$(arg tf_prefix)"/>
     </xacro:include>

File: mur205_description/urdf/ur5_robot.urdf.xacro (robot description, xacro)
@@ -8,5 +8,5 @@
   <!-- <xacro:include filename="$(find ur_description)/urdf/common.gazebo.xacro" /> -->
   <!-- include of the xacro file -->
-  <xacro:include filename="$(find mir_ur5_description)/urdf/ur5.urdf.xacro" />
+  <xacro:include filename="$(find mur205_description)/urdf/ur5.urdf.xacro" />
   <!-- arm -->
   <xacro:ur5_robot prefix="$(arg tf_prefix)" joint_limited="false" transmission_hw_interface="$(arg transmission_hw_interface)"/>
